File: kicad/optojig.sch (KiCad schematic (older format))
At the start: 14 parts

Commit message: Added PCB layout and datasheets
Parts:
- removed D?: LED, symbol LED
- removed R?: R, symbol R
- added BT?: Battery_Cell, symbol Battery_Cell
- added D2: LED, optojig-footprints:TerminalBlock_Buchanan_2way, symbol LED-RESCUE-optojig
- added D?: D, Resistors_ThroughHole:Resistor_Horizontal_RM10mm, symbol D
- added Q1, Q2: 2N2219, optojig-footprints:TO-39, symbol 2N2219
- added R6, R? (x2): 1k, Resistors_ThroughHole:Resistor_Horizontal_RM10mm, symbol R
- added SW1: Switch_SPDT_x2, optojig-footprints:SPDT_switch, symbol Switch_SPDT_x2
- BT1: renamed from BT?; footprint (none) -> optojig-footprints:TerminalBlock_Buchanan_2way
- D1: renamed from D?; footprint (none) -> optojig-footprints:TerminalBlock_Buchanan_2way; symbol LED -> LED-RESCUE-optojig
- R1, R4: renamed from R?; footprint Opto-Devices:Resistor_LDR_10x8.5_RM7.6 -> optojig-footprints:TerminalBlock_Buchanan_2way
- R2, R5: renamed from R?; value R -> 680R; footprint (none) -> Resistors_ThroughHole:Resistor_Horizontal_RM10mm
- R3: renamed from R?; value R -> 1k; footprint (none) -> Resistors_ThroughHole:Resistor_Horizontal_RM10mm
- RV1, RV2: renamed from RV?; footprint (none) -> optojig-footprints:Vishay_Trimmer_Through_Hole_2.54mm; symbol POT -> POT-RESCUE-optojig
- U1: renamed from U?; footprint (none) -> optojig-footprints:TRN_1-0510
- U2: renamed from U?; footprint (none) -> optojig-footprints:DIP-8_W7.62mm_LongPads
- gave numbers to parts that had none: 1
Connections:
- net at U2.1: now also R6.2; no longer R3.1
- net GND: now reaches R2.2, R5.2, RV1.3, RV2.3, U1.5 (-V_out), U2.4 (V-), U2.4 (V-)
- net GND: now also Q1.1 (E), Q2.1 (E); no longer D1.1 (K)
- net at R1.1, R4.1, RV1.1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: now also R?.2, R?.2
- net at BT1.2 (-), U1.1 (-V_in): now also BT?.2 (-)
- net at U1.2 (+V_in): now also SW1.1 (A); no longer BT1.1 (+)
- net at R3.2: now also U2.7; no longer D1.2 (A)
- net at RV2.2: now also U2.6 (-); no longer U2.2 (-)
- net at R4.2, R5.1: now also U2.5 (+); no longer U2.3 (+)
- new net: Q2.2 (B), R3.1
- new net: D1.1 (K), Q2.3 (C)
- new net: D1.2 (A), R?.1
- new net: BT1.1 (+), D?.1 (K), SW1.2 (B)
- new net: Q1.2 (B), R6.1
- new net: D2.1 (K), Q1.3 (C)
- new net: D2.2 (A), R?.1
- new net: BT?.1 (+), D?.2 (A)
Other:
- moved on the sheet: BT1, D1, R1, R2, R3, R4, R5, RV1, RV2, U1, U2A
